Commit message: realtime vector 0.3--> 1

File: src/mecanum_robot_description/urdf/mecanum.urdf.xacro (robot description, xacro)
@@ -1,23 +1,22 @@
 <?xml version="1.0"?>
-<robot name="mecanum" xmlns:xacro="http://www.ros.org/wiki/xacro">
+<robot name="omni_manipulator" xmlns:xacro="http://www.ros.org/wiki/xacro">
 	<!--xacro:include filename="$(find omni_manipulator)/urdf/cycloid_gear_mecanum_wheel.urdf.xacro" /!-->
 	<xacro:include filename="$(find mecanum_robot_description)/urdf/mecanum_frame.urdf.xacro" />
+	<xacro:include filename="$(find mecanum_robot_description)/urdf/cycloid_gear_mecanum_wheel.urdf.xacro" />
 	<xacro:include filename="$(find mecanum_robot_description)/urdf/mecanum.gazebo.xacro" />
-	<xacro:include filename="$(find mecanum_left)/urdf/mecanum_left.urdf.xacro" />
-	<xacro:include filename="$(find mecanum_right)/urdf/mecanum_right.urdf.xacro" />
     <xacro:macro name="robot">
 		<xacro:frame/>
-		<xacro:mecanum_wheel_right prefix="front" parent="frame" reflect="true">
+		<xacro:mecanum_wheel prefix="front_R" parent="frame" reflect="true">
 			<origin xyz="0.23 -0.2541 -0.11838" rpy="${-pi/2} 0 0"/> <!--0.0762, 0.2541, x:0.069734-->
-		</xacro:mecanum_wheel_right>
-        <xacro:mecanum_wheel_left prefix="front" parent="frame" reflect="true">
-			<origin xyz="0.23 0.2541 -0.11838" rpy="${pi/2} 0 0"/>
-		</xacro:mecanum_wheel_left>
-		<xacro:mecanum_wheel_left prefix="back" parent="frame" reflect="false">
-			<origin xyz="-0.23 -0.2541 -0.11838" rpy="${-pi/2} 0 0"/> <!--y:-0.2571, 0.2541, x:0.390266-->
-		</xacro:mecanum_wheel_left>
-        <xacro:mecanum_wheel_right prefix="back" parent="frame" reflect="false">
+		</xacro:mecanum_wheel>
+        <xacro:mecanum_wheel prefix="front_L" parent="frame" reflect="false">
+			<origin xyz="0.23 0.2541 -0.11838" rpy="${-pi/2} 0 0"/>
+		</xacro:mecanum_wheel>
+		<xacro:mecanum_wheel prefix="back_R" parent="frame" reflect="false">
+			<origin xyz="-0.23 -0.2541 -0.11838" rpy="${pi/2} 0 0"/> <!--y:-0.2571, 0.2541, x:0.390266-->
+		</xacro:mecanum_wheel>
+        <xacro:mecanum_wheel prefix="back_L" parent="frame" reflect="true">
 			<origin xyz="-0.23 0.2541 -0.11838" rpy="${pi/2} 0 0"/>
-		</xacro:mecanum_wheel_right>
+		</xacro:mecanum_wheel>
 		<xacro:omni_steering/>
    		</xacro:macro>

File: src/mecanum_robot_description/urdf/mecanum_frame.urdf.xacro (robot description, xacro)
@@ -28,7 +28,8 @@
             </visual>
             <collision>
-                <origin xyz="0 0 0" rpy="${pi/2} 0.0 ${-pi/2}"/>
+                <origin xyz="0 0 0" rpy="$0.0 0.0 0.0"/>
                 <geometry>
-                    <mesh filename="package://mecanum_robot_description/meshes/frame_c.stl" scale="0.001 0.001 0.001"/>
+                    <box size="0.64 0.598 0.2"/>
+                    <!--mesh filename="package://omni_manipulator/meshes/frame_c.stl" scale="0.001 0.001 0.001"/!-->
                 </geometry>
             </collision>
