Commit message: 210602

File: src/mecanum_robot_description/urdf/mecanum_frame.urdf.xacro (robot description, xacro)
@@ -34,5 +34,5 @@
             </collision>
             <inertial>
-                <mass value="20.326" /> <!--20.781-->
+                <mass value="20.781" /> <!--20.781-->
                 <origin xyz="0 0 0" rpy="${pi/2} 0.0 ${-pi/2}"/>
                 <inertia ixx="7.973347e-01" ixy="1.934100e-05"  ixz="4.964300e-05"  iyy="1.264450e+00"  iyz="5.698240e-04"  izz="5.376963e-01" />

Commit message: keyboard controler

File: src/mecanum_robot_description/urdf/mecanum_frame.urdf.xacro (robot description, xacro)
@@ -34,7 +34,7 @@
             </collision>
             <inertial>
-                <mass value="20.781" /> <!--20.781-->
+                <mass value="100.781" /> <!--20.781-->
                 <origin xyz="0 0 0" rpy="${pi/2} 0.0 ${-pi/2}"/>
-                <inertia ixx="7.973347e-01" ixy="1.934100e-05"  ixz="4.964300e-05"  iyy="1.264450e+00"  iyz="5.698240e-04"  izz="5.376963e-01" />
+                <inertia ixx="3.9866734999999998" ixy="9.6705e-05"  ixz="0.000248215"  iyy="6.32225"  iyz="0.00284912"  izz="2.6884815" />
             </inertial>
         </link>

Commit message: 211220

File: src/mecanum_robot_description/urdf/mecanum_frame.urdf.xacro (robot description, xacro)
@@ -28,5 +28,5 @@
             </visual>
             <collision>
-                <origin xyz="0 0 0" rpy="$0.0 0.0 0.0"/>
+                <origin xyz="0 0 0" rpy="0.0 0.0 0.0"/>
                 <geometry>
                     <box size="0.64 0.598 0.2"/>

File: src/mecanum_robot_description/urdf/mecanum_left_ver2/mecanum.urdf.xacro (robot description, xacro)
@@ -7,14 +7,14 @@
     <xacro:macro name="robot">
 		<xacro:frame/>
-		<xacro:mecanum_wheel prefix="mecanum_L_front_R" parent="frame" reflect="true">
+		<xacro:mecanum_wheel prefix="mecanum_L_front_R" parent="frame_left" reflect="true">
 			<origin xyz="0.2541 0.23 -0.11838" rpy="${-pi/2} 0 ${pi/2}"/> <!--0.0762, 0.2541, x:0.069734-->
 		</xacro:mecanum_wheel>
-        <xacro:mecanum_wheel prefix="mecanum_L_front_L" parent="frame" reflect="false">
+        <xacro:mecanum_wheel prefix="mecanum_L_front_L" parent="frame_left" reflect="false">
 			<origin xyz="0.2541 -0.23 -0.11838" rpy="${-pi/2} 0 ${pi/2}"/>
 		</xacro:mecanum_wheel>
-		<xacro:mecanum_wheel prefix="mecanum_L_back_R" parent="frame" reflect="false">
+		<xacro:mecanum_wheel prefix="mecanum_L_back_R" parent="frame_left" reflect="false">
 			<origin xyz="-0.2541 0.23 -0.11838" rpy="${pi/2} 0 ${pi/2}"/> <!--y:-0.2571, 0.2541, x:0.390266-->
 		</xacro:mecanum_wheel>
-        <xacro:mecanum_wheel prefix="mecanum_L_back_L" parent="frame" reflect="true">
+        <xacro:mecanum_wheel prefix="mecanum_L_back_L" parent="frame_left" reflect="true">
 			<origin xyz="-0.2541 -0.23 -0.11838" rpy="${pi/2} 0 ${pi/2}"/>
 		</xacro:mecanum_wheel>

File: src/mecanum_robot_description/urdf/mecanum_left_ver2/mecanum_frame.urdf.xacro (robot description, xacro)
@@ -15,7 +15,7 @@
 		  <origin xyz="0 0 ${base_offset}" rpy="0 0 0" /> <!-- ${wheel_radius} property must be defined inside wheel description -->
 		  <parent link="summit_base_footprint"/>
-		  <child link="frame" />
+		  <child link="frame_left" />
 		</joint>
-        <link name="frame">
+        <link name="frame_left">
             <visual>
                 <origin xyz="0.0 0.0 0.0" rpy="${pi/2} 0.0 0"/> <!--xyz="0.0 0.0 0.0" rpy="${pi/2} 0.0 ${-pi/2}" -->
@@ -28,8 +28,7 @@
             </visual>
             <collision>
-                <origin xyz="0 0 0" rpy="$0.0 0.0 0.0"/>
+                <origin xyz="0 0 0" rpy="0.0 0.0 0.0"/>
                 <geometry>
                     <box size="0.64 0.598 0.2"/>
-                    <!--mesh filename="package://omni_manipulator/meshes/frame_c.stl" scale="0.001 0.001 0.001"/!-->
                 </geometry>
             </collision>
@@ -40,5 +39,5 @@
             </inertial>
         </link>
-        <gazebo reference="frame">
+        <gazebo reference="frame_left">
             <mu1 value="1.0"/>
             <mu2 value="1.0"/>
@@ -46,5 +45,5 @@
             <kd value="1.0" />
             <maxVel>0.001</maxVel>
-            <minDepth>0.0001</minDepth>
+            <minDepth>0.001</minDepth>
             <turnGravityOff>false</turnGravityOff>
             <material>Gazebo/White</material>
