Commit message: 210618 tennis_game debuging

File: src/ball_trajectory/urdf/camera_left.urdf (robot description, URDF)
Before this commit: robot camera_left, 3 links, 2 joints
Links:
- removed link base_footprint
- added link world
Joints:
- joint base_joint: parent base_footprint -> world

File: src/ball_trajectory/urdf/camera_right.urdf (robot description, URDF)
Before this commit: robot camera_right, 3 links, 2 joints
Links:
- removed link base_footprint
- added link world
Joints:
- joint base_joint: parent base_footprint -> world

Commit message: 210629 camera setup

File: src/ball_trajectory/urdf/camera_left.urdf (robot description, URDF)
Before this commit: robot camera_left, 3 links, 2 joints
Links:
- removed link camera_link
- added link camera_link_0; collision box size=0.012 0.132 0.020; visual box size=0.1 0.15 0.1
- added link camera_link_1; visual box size=0.1 0.15 0.1
Joints:
- removed joint camera_joint
- added joint camera_joint_0: type fixed, parent body, child camera_link_0, origin xyz=0 0 1 rpy=0 0 2.355
- added joint camera_joint_1: type fixed, parent body, child camera_link_1, origin xyz=0 0 1 rpy=0 0 0.785398

File: src/ball_trajectory/urdf/camera_right.urdf (robot description, URDF)
Before this commit: robot camera_right, 3 links, 2 joints
Links:
- removed link camera_link
- added link camera_link_0; collision box size=0.012 0.132 0.020; visual box size=0.1 0.15 0.1
- added link camera_link_1; visual box size=0.1 0.15 0.1
Joints:
- removed joint camera_joint
- added joint camera_joint_0: type fixed, parent body, child camera_link_0, origin xyz=0 0 1 rpy=0 0 -2.355
- added joint camera_joint_1: type fixed, parent body, child camera_link_1, origin xyz=0 0 1 rpy=0 0 -0.785398
