Commit message: 210705 tennis net

File: src/mecanum_robot_description/urdf/mecanum_left_ver1/mecanum_frame.urdf.xacro (robot description, xacro)
@@ -19,5 +19,5 @@
         <link name="frame">
             <visual>
-                <origin xyz="0.0 0.0 0.0" rpy="${pi/2} 0.0 0"/> <!--xyz="0.0 0.0 0.0" rpy="${pi/2} 0.0 ${-pi/2}" -->
+                <origin xyz="0.0 0.0 0.0" rpy="${pi/2} 0.0 ${-pi/2}"/> <!-- -->
                 <geometry>
                     <mesh filename="package://mecanum_robot_description/meshes/frame_c.stl" scale="0.001 0.001 0.001"/>
