Commit message: 210827_2

File: src/mecanum_robot_description/urdf/mecanum_left_ver1/cycloid_gear_mecanum_wheel.urdf.xacro (robot description, xacro)
@@ -11,12 +11,4 @@
         <xacro:property name="radius" value="0.0762"/>
         <xacro:property name="length" value="0.045"/>
-        <joint name="${prefix}_wheel_joint" type="continuous">
-            <parent link="${parent}"/>
-            <child link="${prefix}_wheel"/>
-            <xacro:insert_block name="origin" />
-            <axis xyz="0 0 -1" rpy="0 0 0" />
-            <limit effort="100" velocity="1000"/>
-            <joint_properties damping="0.0" friction="1.0"/>
-        </joint>
         <link name="${prefix}_wheel">
             <visual>
@@ -59,4 +51,12 @@
             </inertial>
         </link>
+        <joint name="${prefix}_wheel_joint" type="continuous">
+            <parent link="${parent}"/>
+            <child link="${prefix}_wheel"/>
+            <xacro:insert_block name="origin" />
+            <axis xyz="0 0 -1" rpy="0 0 0" />
+            <limit effort="100" velocity="1000"/>
+            <joint_properties damping="0.0" friction="1.0"/>
+        </joint>
         <!-- Transmission is important to link the joints and the controller (see summit_xl_control/config/summit_xl_control.yaml)-->
         <transmission name="${prefix}_wheel_trans">

File: src/mecanum_robot_description/urdf/mecanum_left_ver2/cycloid_gear_mecanum_wheel.urdf.xacro (robot description, xacro)
@@ -11,12 +11,4 @@
         <xacro:property name="radius" value="0.0762"/>
         <xacro:property name="length" value="0.045"/>
-        <joint name="${prefix}_wheel_joint" type="continuous">
-            <parent link="${parent}"/>
-            <child link="${prefix}_wheel"/>
-            <xacro:insert_block name="origin" />
-            <axis xyz="0 0 -1" rpy="0 0 0" />
-            <limit effort="100" velocity="1000"/>
-            <joint_properties damping="0.0" friction="1.0"/>
-        </joint>
         <link name="${prefix}_wheel">
             <visual>
@@ -59,4 +51,12 @@
             </inertial>
         </link>
+        <joint name="${prefix}_wheel_joint" type="continuous">
+            <parent link="${parent}"/>
+            <child link="${prefix}_wheel"/>
+            <xacro:insert_block name="origin" />
+            <axis xyz="0 0 -1" rpy="0 0 0" />
+            <limit effort="100" velocity="1000"/>
+            <joint_properties damping="0.0" friction="1.0"/>
+        </joint>
         <!-- Transmission is important to link the joints and the controller (see summit_xl_control/config/summit_xl_control.yaml)-->
         <transmission name="${prefix}_wheel_trans">

File: src/mecanum_robot_description/urdf/mecanum_left_ver2/mecanum.gazebo.xacro (robot description, xacro)
@@ -4,5 +4,5 @@
 	<gazebo>
 	    <plugin name="omni_steering" filename="libgazebo_ros_planar_move.so">
-	      <commandTopic>mecanum_0_vel</commandTopic>
+	      <commandTopic>mecanum_L_vel</commandTopic>
 	      <odometryTopic>odom</odometryTopic>
 	      <odometryFrame>odom</odometryFrame>
@@ -15,13 +15,15 @@
   </xacro:macro>
   <!-- ros_control plugin -->
+  <xacro:macro name="ros_control" params="">
   <gazebo>
-    <plugin name="gazebo_ros_control" filename="libgazebo_ros_control.so">
+    <plugin name="mecanum_L_control" filename="libgazebo_ros_control.so">
       <controlPeriod>0.001</controlPeriod>
-      <robotNamespace>/mecanum</robotNamespace>
-      <jointName>front_R_wheel_joint, front_L_wheel_joint, back_R_wheel_joint, back_L_wheel_joint </jointName>
+      <robotNamespace>/mecanum_L</robotNamespace>
+      <!--jointName>front_R_wheel_joint, front_L_wheel_joint, back_R_wheel_joint, back_L_wheel_joint </jointName-->
       <robotSimType>gazebo_ros_control/DefaultRobotHWSim</robotSimType>
-      <legacyModeNS>true</legacyModeNS>
+      <!--legacyModeNS>true</legacyModeNS-->
     </plugin>
   </gazebo>
+  </xacro:macro>
   <!--gazebo>
    <plugin name="gazebo_grasp_fix" filename="libgazebo_grasp_fix.so">

File: src/mecanum_robot_description/urdf/mecanum_left_ver2/mecanum.urdf.xacro (robot description, xacro)
@@ -1,4 +1,4 @@
 <?xml version="1.0"?>
-<robot name="omni_manipulator" xmlns:xacro="http://www.ros.org/wiki/xacro">
+<robot name="mecanum_L" xmlns:xacro="http://www.ros.org/wiki/xacro">
 	<!--xacro:include filename="$(find omni_manipulator)/urdf/cycloid_gear_mecanum_wheel.urdf.xacro" /!-->
 	<xacro:include filename="$(find mecanum_robot_description)/urdf/mecanum_left_ver2/mecanum_frame.urdf.xacro" />
@@ -7,18 +7,19 @@
     <xacro:macro name="robot">
 		<xacro:frame/>
-		<xacro:mecanum_wheel prefix="front_R" parent="frame" reflect="true">
+		<xacro:mecanum_wheel prefix="mecanum_L_front_R" parent="frame" reflect="true">
 			<origin xyz="0.2541 0.23 -0.11838" rpy="${-pi/2} 0 ${pi/2}"/> <!--0.0762, 0.2541, x:0.069734-->
 		</xacro:mecanum_wheel>
-        <xacro:mecanum_wheel prefix="front_L" parent="frame" reflect="false">
+        <xacro:mecanum_wheel prefix="mecanum_L_front_L" parent="frame" reflect="false">
 			<origin xyz="0.2541 -0.23 -0.11838" rpy="${-pi/2} 0 ${pi/2}"/>
 		</xacro:mecanum_wheel>
-		<xacro:mecanum_wheel prefix="back_R" parent="frame" reflect="false">
+		<xacro:mecanum_wheel prefix="mecanum_L_back_R" parent="frame" reflect="false">
 			<origin xyz="-0.2541 0.23 -0.11838" rpy="${pi/2} 0 ${pi/2}"/> <!--y:-0.2571, 0.2541, x:0.390266-->
 		</xacro:mecanum_wheel>
-        <xacro:mecanum_wheel prefix="back_L" parent="frame" reflect="true">
+        <xacro:mecanum_wheel prefix="mecanum_L_back_L" parent="frame" reflect="true">
 			<origin xyz="-0.2541 -0.23 -0.11838" rpy="${pi/2} 0 ${pi/2}"/>
 		</xacro:mecanum_wheel>
 		<xacro:omni_steering/>
-   		</xacro:macro>
+		<xacro:ros_control/>
+	</xacro:macro>
 	<xacro:robot/>
 </robot>

File: src/mecanum_robot_description/urdf/mecanum_right_ver2/cycloid_gear_mecanum_wheel_1.urdf.xacro (robot description, xacro)
@@ -11,12 +11,4 @@
         <xacro:property name="radius" value="0.0762"/>
         <xacro:property name="length" value="0.045"/>
-        <joint name="${prefix}_wheel_joint" type="continuous">
-            <parent link="${parent}"/>
-            <child link="${prefix}_wheel"/>
-            <xacro:insert_block name="origin" />
-            <axis xyz="0 0 -1" rpy="0 0 0" />
-            <limit effort="100" velocity="1000"/>
-            <joint_properties damping="0.0" friction="1.0"/>
-        </joint>
         <link name="${prefix}_wheel">
             <visual>
@@ -59,4 +51,12 @@
             </inertial>
         </link>
+        <joint name="${prefix}_wheel_joint" type="continuous">
+            <parent link="${parent}"/>
+            <child link="${prefix}_wheel"/>
+            <xacro:insert_block name="origin" />
+            <axis xyz="0 0 -1" rpy="0 0 0" />
+            <limit effort="100" velocity="1000"/>
+            <joint_properties damping="0.0" friction="1.0"/>
+        </joint>
         <!-- Transmission is important to link the joints and the controller (see summit_xl_control/config/summit_xl_control.yaml)-->
         <transmission name="${prefix}_wheel_trans">

File: src/mecanum_robot_description/urdf/mecanum_right_ver2/mecanum_1.gazebo.xacro (robot description, xacro)
@@ -4,5 +4,5 @@
 	<gazebo>
 	    <plugin name="omni_steering" filename="libgazebo_ros_planar_move.so">
-	      <commandTopic>mecanum_1_vel</commandTopic>
+	      <commandTopic>mecanum_R_vel</commandTopic>
 	      <odometryTopic>odom</odometryTopic>
 	      <odometryFrame>odom</odometryFrame>
@@ -15,13 +15,15 @@
   </xacro:macro>
   <!-- ros_control plugin -->
+  <xacro:macro name="ros_control" params="">
   <gazebo>
-    <plugin name="gazebo_ros_control" filename="libgazebo_ros_control.so">
+    <plugin name="mecanum_R_control" filename="libgazebo_ros_control.so">
       <controlPeriod>0.001</controlPeriod>
-      <robotNamespace>/mecanum_1</robotNamespace>
-      <jointName>front_R_wheel_joint, front_L_wheel_joint, back_R_wheel_joint, back_L_wheel_joint </jointName>
+      <robotNamespace>/mecanum_R</robotNamespace>
+      <!--jointName>mecanum_R_front_R_wheel_joint, mecanum_R_front_L_wheel_joint, mecanum_R_back_L_wheel_joint, mecanum_R_back_R_wheel_joint </jointName-->
       <robotSimType>gazebo_ros_control/DefaultRobotHWSim</robotSimType>
-      <legacyModeNS>true</legacyModeNS>
+      <!--legacyModeNS>true</legacyModeNS-->
     </plugin>
   </gazebo>
+  </xacro:macro>
   <!--gazebo>
    <plugin name="gazebo_grasp_fix" filename="libgazebo_grasp_fix.so">

File: src/mecanum_robot_description/urdf/mecanum_right_ver2/mecanum_1.urdf.xacro (robot description, xacro)
@@ -1,4 +1,4 @@
 <?xml version="1.0"?>
-<robot name="omni_manipulator" xmlns:xacro="http://www.ros.org/wiki/xacro">
+<robot name="mecanum_R" xmlns:xacro="http://www.ros.org/wiki/xacro">
 	<!--xacro:include filename="$(find omni_manipulator)/urdf/cycloid_gear_mecanum_wheel.urdf.xacro" /!-->
 	<xacro:include filename="$(find mecanum_robot_description)/urdf/mecanum_right_ver2/mecanum_frame.urdf.xacro" />
@@ -7,18 +7,19 @@
     <xacro:macro name="robot">
 		<xacro:frame/>
-		<xacro:mecanum_wheel_1 prefix="front_R" parent="frame" reflect="true">
+		<xacro:mecanum_wheel_1 prefix="mecanum_R_front_R" parent="frame" reflect="true">
 			<origin xyz="0.2541 0.23 -0.11838" rpy="${-pi/2} 0 ${pi/2}"/> <!--0.0762, 0.2541, x:0.069734-->
 		</xacro:mecanum_wheel_1>
-        <xacro:mecanum_wheel_1 prefix="front_L" parent="frame" reflect="false">
+        <xacro:mecanum_wheel_1 prefix="mecanum_R_front_L" parent="frame" reflect="false">
 			<origin xyz="0.2541 -0.23 -0.11838" rpy="${-pi/2} 0 ${pi/2}"/>
 		</xacro:mecanum_wheel_1>
-		<xacro:mecanum_wheel_1 prefix="back_R" parent="frame" reflect="false">
+		<xacro:mecanum_wheel_1 prefix="mecanum_R_back_R" parent="frame" reflect="false">
 			<origin xyz="-0.2541 0.23 -0.11838" rpy="${pi/2} 0 ${pi/2}"/> <!--y:-0.2571, 0.2541, x:0.390266-->
 		</xacro:mecanum_wheel_1>
-        <xacro:mecanum_wheel_1 prefix="back_L" parent="frame" reflect="true">
+        <xacro:mecanum_wheel_1 prefix="mecanum_R_back_L" parent="frame" reflect="true">
 			<origin xyz="-0.2541 -0.23 -0.11838" rpy="${pi/2} 0 ${pi/2}"/>
 		</xacro:mecanum_wheel_1>
 		<xacro:omni_steering/>
-   		</xacro:macro>
+		<xacro:ros_control/>
+	</xacro:macro>
 	<xacro:robot/>
 </robot>

Commit message: UPDATE : file structure

File: src/mecanum_robot_description/urdf/mecanum_left_ver1/cycloid_gear_mecanum_wheel.urdf.xacro (robot description, xacro)
@@ -35,5 +35,4 @@
                 <geometry>
                     <cylinder length="${length}" radius="${radius}"/>
-                    <!--mesh filename="package://omni_manipulator/meshes/mecanum_left.stl" scale="0.001 0.001 0.001" /!-->
                 </geometry>
                 </xacro:if>
@@ -41,5 +40,4 @@
                 <geometry>
                     <cylinder length="${length}" radius="${radius}"/>
-                    <!--mesh filename="package://omni_manipulator/meshes/mecanum_right.stl" scale="0.001 0.001 0.001" /!-->
                     </geometry>
                 </xacro:unless>

File: src/mecanum_robot_description/urdf/mecanum_left_ver1/mecanum.gazebo.xacro (robot description, xacro)
@@ -24,21 +24,3 @@
     </plugin>
   </gazebo>
-  <!--gazebo>
-   <plugin name="gazebo_grasp_fix" filename="libgazebo_grasp_fix.so">
-        <arm>
-           <arm_name>omni_manipulator</arm_name>
-           <palm_link> gripper_case  </palm_link>
-           <gripper_link> finger_R </gripper_link>
-           <gripper_link> finger_L </gripper_link>
-           <gripper_link> ... </gripper_link>
-        </arm>
-       <forces_angle_tolerance>100</forces_angle_tolerance>
-       <update_rate>4</update_rate>
-       <grip_count_threshold>4</grip_count_threshold>
-       <max_grip_count>8</max_grip_count>
-       <release_tolerance>0.005</release_tolerance>
-       <disable_collisions_on_attach>false</disable_collisions_on_attach>
-       <contact_topic>__default_topic__</contact_topic>
-    </plugin>
-</gazebo!-->
 </robot>

File: src/mecanum_robot_description/urdf/mecanum_left_ver1/mecanum.urdf.xacro (robot description, xacro)
@@ -1,5 +1,4 @@
 <?xml version="1.0"?>
 <robot name="omni_manipulator" xmlns:xacro="http://www.ros.org/wiki/xacro">
-	<!--xacro:include filename="$(find omni_manipulator)/urdf/cycloid_gear_mecanum_wheel.urdf.xacro" /!-->
 	<xacro:include filename="$(find mecanum_robot_description)/urdf/mecanum_left_ver1/mecanum_frame.urdf.xacro" />
 	<xacro:include filename="$(find mecanum_robot_description)/urdf/mecanum_left_ver1/cycloid_gear_mecanum_wheel.urdf.xacro" />

File: src/mecanum_robot_description/urdf/mecanum_left_ver1/mecanum_frame.urdf.xacro (robot description, xacro)
@@ -2,5 +2,4 @@
 <robot xmlns:xacro="http://www.ros.org/wiki/xacro" name="robot_frame">
     <xacro:macro name="frame">
-        <!--xacro:include filename="$(find mecanum_robot_description)/urdf/omni_manipulator.gazebo.xacro" /!-->
         <xacro:property name="base_offset" value="0.19458"/> <!-- 0.193608 !-->
         <link name="summit_base_footprint">
@@ -13,5 +12,5 @@
 		</link>
 		<joint name="summit_base_footprint_joint" type="fixed">
-		  <origin xyz="0 0 ${base_offset}" rpy="0 0 0" /> <!-- ${wheel_radius} property must be defined inside wheel description -->
+		  <origin xyz="0 0 ${base_offset}" rpy="0 0 0" />
 		  <parent link="summit_base_footprint"/>
 		  <child link="frame" />
@@ -31,5 +30,4 @@
                 <geometry>
                     <box size="0.64 0.598 0.2"/>
-                    <!--mesh filename="package://omni_manipulator/meshes/frame_c.stl" scale="0.001 0.001 0.001"/!-->
                 </geometry>
             </collision>

File: src/mecanum_robot_description/urdf/mecanum_right_ver1/cycloid_gear_mecanum_wheel_1.urdf.xacro (robot description, xacro)
@@ -43,5 +43,4 @@
                 <geometry>
                     <cylinder length="${length}" radius="${radius}"/>
-                    <!--mesh filename="package://omni_manipulator/meshes/mecanum_left.stl" scale="0.001 0.001 0.001" /!-->
                 </geometry>
                 </xacro:if>
@@ -49,5 +48,4 @@
                 <geometry>
                     <cylinder length="${length}" radius="${radius}"/>
-                    <!--mesh filename="package://omni_manipulator/meshes/mecanum_right.stl" scale="0.001 0.001 0.001" /!-->
                     </geometry>
                 </xacro:unless>

File: src/mecanum_robot_description/urdf/mecanum_right_ver1/mecanum_1.gazebo.xacro (robot description, xacro)
@@ -24,21 +24,3 @@
     </plugin>
   </gazebo>
-  <!--gazebo>
-   <plugin name="gazebo_grasp_fix" filename="libgazebo_grasp_fix.so">
-        <arm>
-           <arm_name>omni_manipulator</arm_name>
-           <palm_link> gripper_case  </palm_link>
-           <gripper_link> finger_R </gripper_link>
-           <gripper_link> finger_L </gripper_link>
-           <gripper_link> ... </gripper_link>
-        </arm>
-       <forces_angle_tolerance>100</forces_angle_tolerance>
-       <update_rate>4</update_rate>
-       <grip_count_threshold>4</grip_count_threshold>
-       <max_grip_count>8</max_grip_count>
-       <release_tolerance>0.005</release_tolerance>
-       <disable_collisions_on_attach>false</disable_collisions_on_attach>
-       <contact_topic>__default_topic__</contact_topic>
-    </plugin>
-</gazebo!-->
 </robot>

File: src/mecanum_robot_description/urdf/mecanum_right_ver1/mecanum_1.urdf.xacro (robot description, xacro)
@@ -1,5 +1,4 @@
 <?xml version="1.0"?>
 <robot name="omni_manipulator" xmlns:xacro="http://www.ros.org/wiki/xacro">
-	<!--xacro:include filename="$(find omni_manipulator)/urdf/cycloid_gear_mecanum_wheel.urdf.xacro" /!-->
 	<xacro:include filename="$(find mecanum_robot_description)/urdf/mecanum_right_ver1/mecanum_frame.urdf.xacro" />
 	<xacro:include filename="$(find mecanum_robot_description)/urdf/mecanum_right_ver1/cycloid_gear_mecanum_wheel_1.urdf.xacro" />

File: src/mecanum_robot_description/urdf/mecanum_right_ver1/mecanum_frame.urdf.xacro (robot description, xacro)
@@ -2,5 +2,4 @@
 <robot xmlns:xacro="http://www.ros.org/wiki/xacro" name="robot_frame">
     <xacro:macro name="frame">
-        <!--xacro:include filename="$(find mecanum_robot_description)/urdf/omni_manipulator.gazebo.xacro" /!-->
         <xacro:property name="base_offset" value="0.19458"/> <!-- 0.193608 !-->
         <link name="summit_base_footprint">
@@ -13,5 +12,5 @@
 		</link>
 		<joint name="summit_base_footprint_joint" type="fixed">
-		  <origin xyz="0 0 ${base_offset}" rpy="0 0 0" /> <!-- ${wheel_radius} property must be defined inside wheel description -->
+		  <origin xyz="0 0 ${base_offset}" rpy="0 0 0" />
 		  <parent link="summit_base_footprint"/>
 		  <child link="frame" />
@@ -31,5 +30,4 @@
                 <geometry>
                     <box size="0.64 0.598 0.2"/>
-                    <!--mesh filename="package://omni_manipulator/meshes/frame_c.stl" scale="0.001 0.001 0.001"/!-->
                 </geometry>
             </collision>

File: src/mecanum_robot_description/urdf/mecanum_right_ver3/mecanum_frame.urdf.xacro (robot description, xacro)
@@ -39,5 +39,5 @@
         </link>
         <joint name="camera_body_joint" type="fixed">
-            <origin xyz="0 0 0" rpy="0 0 0" /> <!-- ${wheel_radius} property must be defined inside wheel description -->
+            <origin xyz="0 0 0" rpy="0 0 0" />
             <parent link="frame"/>
             <child link="camera_body" />
