Commit message: 210913

File: src/ball_trajectory/urdf/camera/camera_left_top.urdf (robot description, URDF)
Before this commit: robot camera_left, 3 links, 2 joints
Links:
- link body: geometry collision cylinder length=2 radius=0.05; visual cylinder length=2 radius=0.05
Joints:
- joint camera_joint_0: origin xyz=0 0 3 rpy=0 0.523599 0 -> xyz=0 0 2 rpy=0 0 0

Commit message: estimate landing point

File: src/ball_trajectory/urdf/camera/camera_left_top.urdf (robot description, URDF)
Before this commit: robot camera_left, 3 links, 2 joints
Links:
- link body: geometry collision cylinder length=0.1 radius=0.05; visual cylinder length=0.1 radius=0.05
Joints:
- joint camera_joint_0: origin xyz=0 0 2 rpy=0 0 0 -> xyz=0 0 0.1 rpy=0 0 0
