Commit message: 210706 yolov5 test

File: src/mecanum_robot_description/urdf/mecanum_left_ver2/mecanum.urdf.xacro (robot description, xacro)
@@ -8,14 +8,14 @@
 		<xacro:frame/>
 		<xacro:mecanum_wheel prefix="front_R" parent="frame" reflect="true">
-			<origin xyz="0.23 -0.2541 -0.11838" rpy="${-pi/2} 0 0"/> <!--0.0762, 0.2541, x:0.069734-->
+			<origin xyz="0.2541 0.23 -0.11838" rpy="${-pi/2} 0 ${pi/2}"/> <!--0.0762, 0.2541, x:0.069734-->
 		</xacro:mecanum_wheel>
         <xacro:mecanum_wheel prefix="front_L" parent="frame" reflect="false">
-			<origin xyz="0.23 0.2541 -0.11838" rpy="${-pi/2} 0 0"/>
+			<origin xyz="0.2541 -0.23 -0.11838" rpy="${-pi/2} 0 ${pi/2}"/>
 		</xacro:mecanum_wheel>
 		<xacro:mecanum_wheel prefix="back_R" parent="frame" reflect="false">
-			<origin xyz="-0.23 -0.2541 -0.11838" rpy="${pi/2} 0 0"/> <!--y:-0.2571, 0.2541, x:0.390266-->
+			<origin xyz="-0.2541 0.23 -0.11838" rpy="${pi/2} 0 ${pi/2}"/> <!--y:-0.2571, 0.2541, x:0.390266-->
 		</xacro:mecanum_wheel>
         <xacro:mecanum_wheel prefix="back_L" parent="frame" reflect="true">
-			<origin xyz="-0.23 0.2541 -0.11838" rpy="${pi/2} 0 0"/>
+			<origin xyz="-0.2541 -0.23 -0.11838" rpy="${pi/2} 0 ${pi/2}"/>
 		</xacro:mecanum_wheel>
 		<xacro:omni_steering/>

File: src/mecanum_robot_description/urdf/mecanum_right_ver2/mecanum_1.urdf.xacro (robot description, xacro)
@@ -8,14 +8,14 @@
 		<xacro:frame/>
 		<xacro:mecanum_wheel_1 prefix="front_R" parent="frame" reflect="true">
-			<origin xyz="0.23 -0.2541 -0.11838" rpy="${-pi/2} 0 0"/> <!--0.0762, 0.2541, x:0.069734-->
+			<origin xyz="0.2541 0.23 -0.11838" rpy="${-pi/2} 0 ${pi/2}"/> <!--0.0762, 0.2541, x:0.069734-->
 		</xacro:mecanum_wheel_1>
         <xacro:mecanum_wheel_1 prefix="front_L" parent="frame" reflect="false">
-			<origin xyz="0.23 0.2541 -0.11838" rpy="${-pi/2} 0 0"/>
+			<origin xyz="0.2541 -0.23 -0.11838" rpy="${-pi/2} 0 ${pi/2}"/>
 		</xacro:mecanum_wheel_1>
 		<xacro:mecanum_wheel_1 prefix="back_R" parent="frame" reflect="false">
-			<origin xyz="-0.23 -0.2541 -0.11838" rpy="${pi/2} 0 0"/> <!--y:-0.2571, 0.2541, x:0.390266-->
+			<origin xyz="-0.2541 0.23 -0.11838" rpy="${pi/2} 0 ${pi/2}"/> <!--y:-0.2571, 0.2541, x:0.390266-->
 		</xacro:mecanum_wheel_1>
         <xacro:mecanum_wheel_1 prefix="back_L" parent="frame" reflect="true">
-			<origin xyz="-0.23 0.2541 -0.11838" rpy="${pi/2} 0 0"/>
+			<origin xyz="-0.2541 -0.23 -0.11838" rpy="${pi/2} 0 ${pi/2}"/>
 		</xacro:mecanum_wheel_1>
 		<xacro:omni_steering/>

Commit message: readme update

File: src/mecanum_robot_description/urdf/mecanum_left_ver2/mecanum.urdf.xacro (robot description, xacro)
@@ -1,5 +1,4 @@
 <?xml version="1.0"?>
 <robot name="mecanum_L" xmlns:xacro="http://www.ros.org/wiki/xacro">
-	<!--xacro:include filename="$(find omni_manipulator)/urdf/cycloid_gear_mecanum_wheel.urdf.xacro" /!-->
 	<xacro:include filename="$(find mecanum_robot_description)/urdf/mecanum_left_ver2/mecanum_frame.urdf.xacro" />
 	<xacro:include filename="$(find mecanum_robot_description)/urdf/mecanum_left_ver2/cycloid_gear_mecanum_wheel.urdf.xacro" />

File: src/mecanum_robot_description/urdf/mecanum_left_ver2/mecanum_frame.urdf.xacro (robot description, xacro)
@@ -2,5 +2,4 @@
 <robot xmlns:xacro="http://www.ros.org/wiki/xacro" name="robot_frame">
     <xacro:macro name="frame">
-        <!--xacro:include filename="$(find mecanum_robot_description)/urdf/omni_manipulator.gazebo.xacro" /!-->
         <xacro:property name="base_offset" value="0.19458"/> <!-- 0.193608 !-->
         <link name="summit_base_footprint">
@@ -13,5 +12,5 @@
 		</link>
 		<joint name="summit_base_footprint_joint" type="fixed">
-		  <origin xyz="0 0 ${base_offset}" rpy="0 0 0" /> <!-- ${wheel_radius} property must be defined inside wheel description -->
+		  <origin xyz="0 0 ${base_offset}" rpy="0 0 0" />
 		  <parent link="summit_base_footprint"/>
 		  <child link="frame_left" />

File: src/mecanum_robot_description/urdf/mecanum_right_ver2/mecanum_1.urdf.xacro (robot description, xacro)
@@ -1,5 +1,4 @@
 <?xml version="1.0"?>
 <robot name="mecanum_R" xmlns:xacro="http://www.ros.org/wiki/xacro">
-	<!--xacro:include filename="$(find omni_manipulator)/urdf/cycloid_gear_mecanum_wheel.urdf.xacro" /!-->
 	<xacro:include filename="$(find mecanum_robot_description)/urdf/mecanum_right_ver2/mecanum_frame.urdf.xacro" />
 	<xacro:include filename="$(find mecanum_robot_description)/urdf/mecanum_right_ver2/cycloid_gear_mecanum_wheel_1.urdf.xacro" />

File: src/mecanum_robot_description/urdf/mecanum_right_ver2/mecanum_frame.urdf.xacro (robot description, xacro)
@@ -2,5 +2,4 @@
 <robot xmlns:xacro="http://www.ros.org/wiki/xacro" name="robot_frame">
     <xacro:macro name="frame">
-        <!--xacro:include filename="$(find mecanum_robot_description)/urdf/omni_manipulator.gazebo.xacro" /!-->
         <xacro:property name="base_offset" value="0.19458"/> <!-- 0.193608 !-->
         <link name="summit_base_footprint">
@@ -13,5 +12,5 @@
 		</link>
 		<joint name="summit_base_footprint_joint" type="fixed">
-		  <origin xyz="0 0 ${base_offset}" rpy="0 0 0" /> <!-- ${wheel_radius} property must be defined inside wheel description -->
+		  <origin xyz="0 0 ${base_offset}" rpy="0 0 0" />
 		  <parent link="summit_base_footprint"/>
 		  <child link="frame" />

File: src/mecanum_robot_description/urdf/mecanum_right_ver3/mecanum_1.urdf.xacro (robot description, xacro)
@@ -1,5 +1,4 @@
 <?xml version="1.0"?>
 <robot name="mecanum_R" xmlns:xacro="http://www.ros.org/wiki/xacro">
-	<!--xacro:include filename="$(find omni_manipulator)/urdf/cycloid_gear_mecanum_wheel.urdf.xacro" /!-->
 	<xacro:include filename="$(find mecanum_robot_description)/urdf/mecanum_right_ver3/mecanum_frame.urdf.xacro" />
 	<xacro:include filename="$(find mecanum_robot_description)/urdf/mecanum_right_ver3/cycloid_gear_mecanum_wheel_1.urdf.xacro" />

File: src/mecanum_robot_description/urdf/mecanum_right_ver3/mecanum_frame.urdf.xacro (robot description, xacro)
@@ -2,5 +2,4 @@
 <robot xmlns:xacro="http://www.ros.org/wiki/xacro" name="robot_frame">
     <xacro:macro name="frame">
-        <!--xacro:include filename="$(find mecanum_robot_description)/urdf/omni_manipulator.gazebo.xacro" /!-->
         <xacro:property name="base_offset" value="0.19458"/> <!-- 0.193608 !-->
         <link name="summit_base_footprint">
@@ -13,5 +12,5 @@
 		</link>
 		<joint name="summit_base_footprint_joint" type="fixed">
-		  <origin xyz="0 0 ${base_offset}" rpy="0 0 0" /> <!-- ${wheel_radius} property must be defined inside wheel description -->
+		  <origin xyz="0 0 ${base_offset}" rpy="0 0 0" />
 		  <parent link="summit_base_footprint"/>
 		  <child link="frame" />
