Commit message: UPDATE: add catch net stl && update yolov5 version && mecanum ver2 camera

File: src/mecanum_robot_description/urdf/mecanum_left_ver2/mecanum_frame.urdf.xacro (robot description, xacro)
@@ -38,4 +38,65 @@
             </inertial>
         </link>
+        <joint name="camera_body_joint" type="fixed">
+            <origin xyz="0 0 0.05" rpy="0 0 0" />
+            <parent link="frame_left"/>
+            <child link="camera_body" />
+        </joint>
+        <link name="camera_body">
+            <inertial>
+                <origin
+                    xyz="0 0 0.35"
+                    rpy="0 0 0" />
+                <mass
+                    value="3" />
+                <inertia
+                    ixx="0.003958333"
+                    ixy="0"
+                    ixz="0"
+                    iyy="0.003958333"
+                    iyz="0"
+                    izz="0.02" />
+            </inertial>
+            <visual>
+                <origin
+                    xyz="0.0 0 0.35"
+                    rpy="0 0 0" />
+                <geometry>
+                    <cylinder length="0.8" radius="0.05"/>
+                </geometry>
+                <material
+                    name="">
+                    <color
+                    rgba="0.84706 0.83922 0.83922 1" />
+                </material>
+            </visual>
+            <collision>
+                <origin
+                    xyz="0.0 0 0.35"
+                    rpy="0 0 0" />
+                <geometry>
+                    <cylinder length="0.8" radius="0.05"/>
+                </geometry>
+            </collision>
+        </link> -->
+        <joint name="camera_joint_0" type="fixed">
+            <origin xyz="0.0 0 0.80542" rpy="0 0 0"/>
+            <parent link="frame_left"/>
+            <child link="camera_link"/>
+        </joint>
+        <link name="camera_link">
+            <visual>
+                <origin xyz="0. 0 0" rpy="0 0 0"/>
+                <geometry>
+                    <box size="0.1 0.2 0.1" />
+                </geometry>
+            </visual>
+            <collision>
+                <origin xyz="0. 0 0" rpy="0 0 0"/>
+                <geometry>
+                    <box size="0.1 0.2 0.1" />
+                </geometry>
+            </collision>
+        </link>
         <gazebo reference="frame_left">
             <mu1 value="1.0"/>

File: src/mecanum_robot_description/urdf/mecanum_right_ver2/mecanum_1.gazebo.xacro (robot description, xacro)
@@ -25,4 +25,46 @@
     </plugin>
   </gazebo>
+  <gazebo reference="camera_link">
+      <sensor name="mecanum_camera_ir" type="depth">
+        <update_rate>60</update_rate>
+        <camera>
+          <horizontal_fov>1.5708</horizontal_fov>
+          <vertical_fov>1.02974</vertical_fov>
+          <image>
+            <width>640</width>
+            <height>360</height>
+            <format>R8G8B8</format>
+          </image>
+          <clip>
+            <near>0.1</near>
+            <far>30</far>
+          </clip>
+        </camera>
+        <plugin name="mecanum_camera_ir_controller" filename="libgazebo_ros_openni_kinect.so">
+          <baseline>0.1</baseline>
+          <alwaysOn>false</alwaysOn>
+          <update_rate>60</update_rate>
+          <cameraName>mecanum_camera_ir</cameraName>
+          <imageTopicName>mecanum_camera_ir/color/image_raw</imageTopicName>
+          <cameraInfoTopicName>/mecanum_camera_ir/color/camera_info</cameraInfoTopicName>
+          <depthImageTopicName>/mecanum_camera_ir/depth/image_raw</depthImageTopicName>
+          <depthImageInfoTopicName>/mecanum_camera_ir/depth/camera_info</depthImageInfoTopicName>
+          <pointCloudTopicName>/mecanum_camera_ir/depth/points</pointCloudTopicName>
+          <frameName>camera_link</frameName>
+          <pointCloudCutoff>0.1</pointCloudCutoff>
+          <pointCloudCutoffMax>15.0</pointCloudCutoffMax>
+          <distortionK1>0.00000001</distortionK1>
+          <distortionK2>0.00000001</distortionK2>
+          <distortionK3>0.00000001</distortionK3>
+          <distortionT1>0.00000001</distortionT1>
+          <distortionT2>0.00000001</distortionT2>
+          <!-- <CxPrime>0</CxPrime>
+          <Cx>640</Cx>
+          <Cy>360</Cy>
+          <focalLength>639.9976491530514</focalLength> -->
+          <hackBaseline>0</hackBaseline>
+        </plugin>
+      </sensor>
+    </gazebo>
   </xacro:macro>
   <!--gazebo>

File: src/mecanum_robot_description/urdf/mecanum_right_ver2/mecanum_frame.urdf.xacro (robot description, xacro)
@@ -39,4 +39,65 @@
             </inertial>
         </link>
+        <joint name="camera_body_joint" type="fixed">
+            <origin xyz="0 0 0.05" rpy="0 0 0" />
+            <parent link="frame"/>
+            <child link="camera_body" />
+        </joint>
+        <link name="camera_body">
+            <inertial>
+                <origin
+                    xyz="0 0 0.35"
+                    rpy="0 0 0" />
+                <mass
+                    value="3" />
+                <inertia
+                    ixx="0.003958333"
+                    ixy="0"
+                    ixz="0"
+                    iyy="0.003958333"
+                    iyz="0"
+                    izz="0.02" />
+            </inertial>
+            <visual>
+                <origin
+                    xyz="0.0 0 0.35"
+                    rpy="0 0 0" />
+                <geometry>
+                    <cylinder length="0.8" radius="0.05"/>
+                </geometry>
+                <material
+                    name="">
+                    <color
+                    rgba="0.84706 0.83922 0.83922 1" />
+                </material>
+            </visual>
+            <collision>
+                <origin
+                    xyz="0.0 0 0.35"
+                    rpy="0 0 0" />
+                <geometry>
+                    <cylinder length="0.8" radius="0.05"/>
+                </geometry>
+            </collision>
+        </link> -->
+        <joint name="camera_joint_0" type="fixed">
+            <origin xyz="0.0 0 0.80542" rpy="0 0 0"/>
+            <parent link="frame"/>
+            <child link="camera_link"/>
+        </joint>
+        <link name="camera_link">
+            <visual>
+                <origin xyz="0. 0 0" rpy="0 0 0"/>
+                <geometry>
+                    <box size="0.1 0.2 0.1" />
+                </geometry>
+            </visual>
+            <collision>
+                <origin xyz="0. 0 0" rpy="0 0 0"/>
+                <geometry>
+                    <box size="0.1 0.2 0.1" />
+                </geometry>
+            </collision>
+        </link>
         <gazebo reference="frame">
             <mu1 value="1.0"/>
