Commit message: ADD: Tennis robot catch ball based robot camera

File: src/mecanum_robot_description/urdf/mecanum_right_ver3/mecanum_frame.urdf.xacro (robot description, xacro)
@@ -41,59 +41,59 @@
             <origin xyz="0 0 0" rpy="0 0 0" />
             <parent link="frame"/>
-            <child link="camera_body" />
+            <child link="tennis_robot_net" />
           </joint>
-        <link name="camera_body">
+        <link name="tennis_robot_net">
             <inertial>
-            <origin
-                xyz="0 0 0.4"
-                rpy="0 0 0" />
-            <mass
-                value="1" />
-            <inertia
-                ixx="0.003958333"
-                ixy="0"
-                ixz="0"
-                iyy="0.003958333"
-                iyz="0"
-                izz="0.02" />
+                <origin
+                    xyz="0.15 0 -0.1"
+                    rpy="0 0 0" />
+                <mass
+                    value="1" />
+                <inertia
+                    ixx="0.003958333"
+                    ixy="0"
+                    ixz="0"
+                    iyy="0.003958333"
+                    iyz="0"
+                    izz="0.02" />
             </inertial>
             <visual>
-            <origin
-                xyz="0 0 0.4"
-                rpy="0 0 0" />
-            <geometry>
-                <cylinder length="0.8" radius="0.05"/>
-            </geometry>
-            <material
-                name="">
-                <color
-                rgba="0.84706 0.83922 0.83922 1" />
-            </material>
+                <origin
+                    xyz="0.15 0 -0.1"
+                    rpy="0 0 0" />
+                <geometry>
+                    <mesh filename="package://mecanum_robot_description/meshes/tennis_robot_net1.stl" scale="0.001 0.001 0.001"/>
+                </geometry>
+                <material
+                    name="">
+                    <color
+                    rgba="0.84706 0.83922 0.83922 1" />
+                </material>
             </visual>
             <collision>
-            <origin
-                xyz="0 0 0.4"
-                rpy="0 0 0" />
-            <geometry>
-                <cylinder length="0.8" radius="0.05"/>
-            </geometry>
+                <origin
+                    xyz="0.15 0 -0.1"
+                    rpy="0 0 0" />
+                <geometry>
+                    <mesh filename="package://mecanum_robot_description/meshes/tennis_robot_net1.stl" scale="0.001 0.001 0.001"/>
+                </geometry>
             </collision>
-            </link>
+        </link>
         <joint name="camera_joint_0" type="fixed">
-            <origin xyz="0 0 0.8" rpy="0 0 0"/>
-            <parent link="camera_body"/>
+            <origin xyz="0.1 0 0.75" rpy="0 0 0"/>
+            <parent link="tennis_robot_net"/>
             <child link="camera_link"/>
         </joint>
         <link name="camera_link">
             <visual>
-                <origin xyz="0 0 0" rpy="0 0 0"/>
+                <origin xyz="0.1 0 0" rpy="0 0 0"/>
                 <geometry>
-                    <box size="0.1 0.2 0.1" />
+                    <box size="0.03 0.2 0.1" />
                 </geometry>
             </visual>
             <collision>
-                <origin xyz="0.0 0.0 0.0" rpy="0 0 0"/>
+                <origin xyz="0.1 0 0" rpy="0 0 0"/>
                 <geometry>
-                    <box size="0.1 0.2 0.1" />
+                    <box size="0.03 0.2 0.1" />
                 </geometry>
             </collision>
@@ -108,4 +108,14 @@
             <turnGravityOff>false</turnGravityOff>
             <material>Gazebo/White</material>
+        </gazebo>
+        <gazebo reference="tennis_robot_net">
+            <mu1 value="1.0"/>
+            <mu2 value="1.0"/>
+            <kp>100000000</kp>
+            <kd>100000000</kd>
+            <max_vel>0</max_vel>
+            <min_depth>0</min_depth>
+            <turnGravityOff>false</turnGravityOff>
+            <material>Gazebo/grey</material>
         </gazebo>
         <gazebo reference="camera_link">

Commit message: EDIT: mecanum catch ball code

File: src/mecanum_robot_description/urdf/mecanum_right_ver3/mecanum_frame.urdf.xacro (robot description, xacro)
@@ -46,5 +46,5 @@
             <inertial>
                 <origin
-                    xyz="0.15 0 -0.1"
+                    xyz="0.15 0 0.585"
                     rpy="0 0 0" />
                 <mass
@@ -60,8 +60,8 @@
             <visual>
                 <origin
-                    xyz="0.15 0 -0.1"
+                    xyz="0.15 0 0.585"
                     rpy="0 0 0" />
                 <geometry>
-                    <mesh filename="package://mecanum_robot_description/meshes/tennis_robot_net1.stl" scale="0.001 0.001 0.001"/>
+                    <mesh filename="package://mecanum_robot_description/meshes/net500x450.stl" scale="0.01 0.01 0.01"/>
                 </geometry>
                 <material
@@ -73,14 +73,14 @@
             <collision>
                 <origin
-                    xyz="0.15 0 -0.1"
+                    xyz="0.15 0 0.585"
                     rpy="0 0 0" />
                 <geometry>
-                    <mesh filename="package://mecanum_robot_description/meshes/tennis_robot_net1.stl" scale="0.001 0.001 0.001"/>
+                    <mesh filename="package://mecanum_robot_description/meshes/net500x450.stl" scale="0.01 0.01 0.01"/>
                 </geometry>
             </collision>
         </link>
         <joint name="camera_joint_0" type="fixed">
-            <origin xyz="0.1 0 0.75" rpy="0 0 0"/>
-            <parent link="tennis_robot_net"/>
+            <origin xyz="0.05 0 1.02" rpy="0 0 0"/>
+            <parent link="frame"/>
             <child link="camera_link"/>
         </joint>

Commit message: ADD: tennis robot net part

File: src/mecanum_robot_description/urdf/mecanum_right_ver3/mecanum_frame.urdf.xacro (robot description, xacro)
@@ -49,5 +49,5 @@
                     rpy="0 0 0" />
                 <mass
-                    value="1" />
+                    value="8" />
                 <inertia
                     ixx="0.003958333"
@@ -63,5 +63,5 @@
                     rpy="0 0 0" />
                 <geometry>
-                    <mesh filename="package://mecanum_robot_description/meshes/net500x450.stl" scale="0.01 0.01 0.01"/>
+                    <mesh filename="package://mecanum_robot_description/meshes/net450x450.stl" scale="0.001 0.001 0.001"/>
                 </geometry>
                 <material
@@ -76,5 +76,5 @@
                     rpy="0 0 0" />
                 <geometry>
-                    <mesh filename="package://mecanum_robot_description/meshes/net500x450.stl" scale="0.01 0.01 0.01"/>
+                    <mesh filename="package://mecanum_robot_description/meshes/net450x450.stl" scale="0.001 0.001 0.001"/>
                 </geometry>
             </collision>

Commit message: ADD: net camera test data

File: src/mecanum_robot_description/urdf/mecanum_right_ver3/mecanum_frame.urdf.xacro (robot description, xacro)
@@ -38,10 +38,10 @@
             </inertial>
         </link>
-        <joint name="camera_body_joint" type="fixed">
+        <!--<joint name="camera_body_joint" type="fixed">
             <origin xyz="0 0 0" rpy="0 0 0" />
             <parent link="frame"/>
             <child link="tennis_robot_net" />
           </joint>
-        <link name="tennis_robot_net">
+         <link name="tennis_robot_net">
             <inertial>
                 <origin
@@ -79,5 +79,5 @@
                 </geometry>
             </collision>
-        </link>
+        </link> -->
         <joint name="camera_joint_0" type="fixed">
             <origin xyz="0.05 0 1.02" rpy="0 0 0"/>
